File: Pure VCF.sch (EAGLE design)
At the start: 82 parts, among them T1 TRANS_PAIR_PNP, U1 QUAD_OPAMP, U2 LM13700, U3 DUAL_OPAMP, U4 LM13700

Commit message: VCF 2.2
Parts:
- C10, C11, C12, C9: value 100nF -> 0.1u; device rcl:C-USC1206K -> rcl:C-USC0805K
- C14, C15, C16, C17: value * -> 0.1u
- R21: value 300K -> 75K***
- R22: value 49K9 -> 1M***
- R23: value 100K -> 4k12
- R3: value 100K -> 1M***
- R39: value 2K2 -> 4k12
- R4: value 100K -> 1M5***
- R6: value 220K -> 2M***
- R7: value 2K2 -> 0R***
- TR1: value 100R -> 100K; device INSTRUO:TRIM_3269W -> INSTRUO:TRIMMER_TH3
- TR2: value 100R -> 100k
Connections:
- net -12V: now also R21.1; no longer COF.1
- net GND: now also R22.2; no longer U1G$1.+IN
- net N$19: now also R23.1; no longer R22.1
- net N$20: now also Q.3, U1G$1.OUT; no longer R21.1, R22.2
- net N$25: now also COF.1; no longer R23.1, U1G$1.OUT
- net N$46: now also U1G$1.+IN; no longer Q.3
- net N$7: now also R22.1
Other:
- note added: "0R"
- note added: "2M"
- moved on the sheet: C10, C11, C12, C14, C15, C16, C17, C9, R21, R22

Commit message: VCF 2.3
Parts:
- removed R22: 1M***, rcl:R-US_R0805
- removed R5: 220K, rcl:R-US_R0805
- removed U1: QUAD_OPAMP, INSTRUO:QUAD_OPAMP
- removed U2, U4: LM13700, INSTRUO:LM13700
- removed U3: DUAL_OPAMP, INSTRUO:DUAL_OPAMP
- added IC4, IC5: TL074D, GMSN:TL074D
- added U$3, U$4: LM13700, GMSN:LM13700
- 2POLE, 4POLE, COF_CV: device INSTRUO:S_JACK -> GMSN:S_JACK
- C13, C8: device rcl:CPOL-US153CLV-0505 -> GMSN:CPOL-US153CLV-0505
- C3: device rcl:C-USC0805K -> GMSN:C-USC0805K
- C4, C5, C6, C7: device rcl:C-USC0805K -> rcl:C-US050-045X075
- COF, CV_AT, IN1POT, IN1POT1: device INSTRUO:Q-POT -> GMSN:9MMPOT
- Q: value 100K -> 100k; device INSTRUO:Q-POT -> GMSN:9MMPOT
- R0: value 2K -> 2k
- R1, R10, R13, R15, R18, R26, R30, R31, R34, R41, R43, R44, R8: value 100K -> 100k; device rcl:R-US_R0805 -> GMSN:R-US_R0805
- R11, R20, R28, R42: value 33K -> 33k; device rcl:R-US_R0805 -> GMSN:R-US_R0805
- R12, R16, R17, R2, R27, R29, R33, R36, R6, R9: device rcl:R-US_R0805 -> GMSN:R-US_R0805
- R14, R32, R35: value 10K -> 10k; device rcl:R-US_R0805 -> GMSN:R-US_R0805
- R19: value 100K -> 10k; device rcl:R-US_R0805 -> GMSN:R-US_R0805
- R21: value 75K*** -> 75k
- R23: value 4k12 -> 10k; device rcl:R-US_R0805 -> GMSN:R-US_R0805
- R24, R25, R37, R38, R40: value 2K2 -> 100k; device rcl:R-US_R0805 -> GMSN:R-US_R0805
- R3: value 1M*** -> 100k; device rcl:R-US_R0805 -> GMSN:R-US_R0805
- R39: value 4k12 -> 100k; device rcl:R-US_R0805 -> GMSN:R-US_R0805
- R4: value 1M5*** -> 100k; device rcl:R-US_R0805 -> GMSN:R-US_R0805
- R7: value 0R*** -> 2k2; device rcl:R-US_R0805 -> GMSN:R-US_R0805
- T1: device INSTRUO:TRANS_PAIR_PNP -> GMSN:TRANS_PAIR_PNP
- TR1: value 100K -> 100k; device INSTRUO:TRIMMER_TH3 -> GMSN:TRIMMER_TH3
- TR2: value 100k -> TRIMMER_TH3; device INSTRUO:TRIM_3269W -> GMSN:TRIMMER_TH3
Connections:
- removed net N$34: R29.1, R30.1, U4G$1.IN-
- removed net N$42: R41.2, R43.1, R44.1, U1G$2.-IN
- removed net N$45: C7.1, U4G$2.OUT, U4G$4.BUF-IN_2
- removed net N$48: R42.1, U4G$2.BIAS-IN
- removed net N$51: U4G$1.D-BIAS
- removed net N$52: U4G$2.D-BIAS
- new net N$57: C6.1, U$4G$1.BUF-IN_2, U$4G$1.OUT
- new net N$58: C7.1, U$4G$2.BUF-IN_2, U$4G$2.OUT
- new net N$59: R28.1, U$4G$1.BIAS-IN
- net +12V: now also IC4P.V+, IC5P.V+, U$3G$3.V++, U$4G$3.V++; no longer U1G$5.+12V, U2G$3.V++, U3G$3.+12V, U4G$3.V++
- net -12V: now also IC4P.V-, IC5P.V-, U$3G$3.V--, U$4G$3.V--; no longer U1G$6.-12V, U2G$3.V--, U3G$4.-12V, U4G$3.V--
- net GND: now also IC4A.+IN, IC4B.+IN, IC4C.+IN, IC5A.+IN, IC5B.+IN, IC5D.+IN; no longer R22.2, R5.1, U1G$2.+IN, U3G$1.+IN, U3G$2.+IN
- net N$1: now also C5.1, U$3G$2.BUF-IN_2, U$3G$2.OUT; no longer U2G$1.D-BIAS
- net N$11: now also IC4A.-IN; no longer U1G$4.-IN
- net N$12: now also IC4A.OUT; no longer U1G$4.OUT
- net N$13: now also U$3G$1.BIAS-IN; no longer U2G$1.BIAS-IN
- net N$15: now also IC4B.-IN, R41.2, R43.1, R44.1; no longer R5.2, U1G$4.+IN
- net N$16: now also U$3G$2.BUF-OUT_2; no longer U2G$4.BUF-OUT_2
- net N$17: now also U$3G$1.IN+; no longer U2G$1.IN+
- net N$18: now also C8.-, IC5A.-IN, R40.1; no longer R10.1, R12.1, R13.1, R23.2, U2G$1.IN-
- net N$20: now also IC5C.-IN, IC5C.OUT; no longer U1G$1.-IN, U1G$1.OUT
- net N$21: now also C13.-, IC5B.-IN, R39.1; no longer C8.-, R40.1, U3G$2.-IN
- net N$22: now also U$3G$2.BIAS-IN; no longer U2G$2.BIAS-IN
- net N$23: now also U$3G$2.IN+; no longer U2G$2.IN+
- net N$24: now also U$3G$2.IN-; no longer U2G$2.IN-
- net N$27: now also U$3G$1.BUF-IN_2, U$3G$1.OUT; no longer U2G$1.OUT, U2G$4.BUF-IN_1
- net N$28: now also U$3G$1.BUF-OUT_2; no longer U2G$4.BUF-OUT_1
- net N$29: now also R26.1, R27.1, U$4G$1.IN+; no longer C5.1, U2G$2.OUT, U2G$4.BUF-IN_2
- net N$30: now also IC5A.OUT; no longer U3G$2.OUT
- net N$31: now also R42.1, U$4G$2.BIAS-IN; no longer R28.1, U4G$1.BIAS-IN
- net N$32: now also IC4B.OUT; no longer U1G$2.OUT
- net N$33: now also R29.1, R30.1, U$4G$1.IN-; no longer R26.1, R27.1, U4G$1.IN+
- net N$37: now also IC5D.-IN, IC5D.OUT; no longer C13.-, R39.1, U3G$1.-IN
- net N$39: now also IC4C.-IN, IC4C.OUT; no longer R31.1, R33.1, U4G$2.IN+
- net N$4: now also R10.1, R12.1, R13.1, R23.2, U$3G$1.IN-; no longer U2G$2.D-BIAS
- net N$40: now also U$4G$2.IN-; no longer U4G$2.IN-
- net N$41: now also IC5B.OUT; no longer U3G$1.OUT
- net N$43: now also R31.1, R33.1, U$4G$2.IN+; no longer C6.1, U4G$1.OUT, U4G$4.BUF-IN_1
- net N$44: now also U$4G$1.BUF-OUT_2; no longer U4G$4.BUF-OUT_1
- net N$46: now also IC5C.+IN, U$4G$2.BUF-OUT_2; no longer U1G$1.+IN, U4G$4.BUF-OUT_2
- net N$5: now also IC4D.OUT; no longer U1G$3.OUT
- net N$6: now also IC4D.-IN; no longer U1G$3.-IN
- net N$7: no longer R22.1
- net N$8: now also IC4D.+IN; no longer U1G$3.+IN
Other:
- note added: "Maximum output current: Negative Saturation Voltage/ R7 = 5.4mA"
- note added: "R2 can be lowered if V/Oct range is too high. 100R min."
- note added: "Ray Wilson had matched PNPs at each stage"
- note added: "Reduce the current limiting resistors to raise the top end of the cutoff. 7.5k min"
- note added: "Reference current: Iref=Vsupply/R = 6uA"
- note removed: "0R"
- note removed: "2M"
- moved on the sheet: 2POLE, 4POLE, C1, C10, C11, C12, C14, C15, C16, C17, C2, C4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

Commit message: VCF 2.4
Parts:
- removed IC5: TL074D, GMSN:TL074D
- removed R0: 2k, INSTRUO:R_TC
- removed R44: 100k, GMSN:R-US_R0805
- removed U$3, U$4: LM13700, GMSN:LM13700
- added IC1, IC2: LM13700, GMSN:OTA_LM13700
- added IC3: TL074, GMSN:OPAMP_QUADD
- added R22: 100k, GMSN:RESISTOR_USR0805
- added R5: Tempco 2k, GMSN:RESISTOR_US0204/7
- 2POLE, 4POLE, COF_CV: value S_JACK -> PJ301M-12; device GMSN:S_JACK -> GMSN:SOCKET_MONO_3.5MMPJ301M-12
- C1, C2: value 10u -> 10uF; device rcl:CPOL-US153CLV-0505 -> GMSN:CAPACITOR_POL-US153CLV-0505
- C10, C11, C12, C14, C15, C16, C17, C9: value 0.1u -> 100nF; device rcl:C-USC0805K -> GMSN:CAPACITOR-USC0805
- C13, C8: value 10u -> 10uF; device GMSN:CPOL-US153CLV-0505 -> GMSN:CAPACITOR_POL-US153CLV-0505
- C3: value 20pF -> 22pF; device GMSN:C-USC0805K -> GMSN:CAPACITOR-USC0805
- C4, C5, C6, C7: device rcl:C-US050-045X075 -> GMSN:CAPACITOR-US050-045X075
- COF, CV_AT, IN1POT, IN1POT1: value 100K -> 100k; device GMSN:9MMPOT -> GMSN:RESISTOR_VARIABLE9MM_POT
- D1, D2: value (none) -> STTH102A; device adafruit:DIODESMA -> GMSN:DIODESMA
- IC4: value TL074D -> TL074; device GMSN:TL074D -> GMSN:OPAMP_QUADD
- IN1, IN2: value S_JACK -> PJ301M-12; device INSTRUO:S_JACK -> GMSN:SOCKET_MONO_3.5MMPJ301M-12
- JP1: value M05X2SHD -> HEADER2X5SHD; device SparkFun-Connectors:M05X2SHD -> GMSN:HEADER2X5SHD
- Q: device GMSN:9MMPOT -> GMSN:RESISTOR_VARIABLE9MM_POT
- R1, R10, R11, R12, R13, R14, R15, R16, R17, R18, R19, R2, R20, R23, R24, R25, R26, R27, R28, R29, R3, R30, R31, R32, R33, R34, R35, R36, R37, R38, R39, R4, R40, R41, R42, R43, R7, R8, R9: device GMSN:R-US_R0805 -> GMSN:RESISTOR_USR0805
- R21: device rcl:R-US_R0805 -> GMSN:RESISTOR_USR0805
- R6: value 2M*** -> 2M; device GMSN:R-US_R0805 -> GMSN:RESISTOR_USR0805
- T1: value TRANS_PAIR_PNP -> DMMT3906W; device GMSN:TRANS_PAIR_PNP -> GMSN:TRANSISTOR_PAIR_PNP
- TR1: device GMSN:TRIMMER_TH3 -> GMSN:RESISTOR_VARIABLETRIMMER_TH
- TR2: value TRIMMER_TH3 -> 100k; device GMSN:TRIMMER_TH3 -> GMSN:RESISTOR_VARIABLETRIMMER_TH
Connections:
- net +12V: now also IC1G$3.V+, IC2G$3.V+, IC3P.V+; no longer IC5P.V+, U$3G$3.V++, U$4G$3.V++
- net -12V: now also IC1G$3.V-, IC2G$3.V-, IC3P.V-; no longer IC5P.V-, U$3G$3.V--, U$4G$3.V--
- net GND: now also 2POLE.SLEEVE, 4POLE.SLEEVE, COF_CV.SLEEVE, COF_CV.SWITCH, IC3A.+IN, IC3B.+IN, IC3D.+IN, IN1.SLEEVE, IN2.SLEEVE; no longer 2POLE.GND, 4POLE.GND, COF_CV.GND, COF_CV.NORM, IC5A.+IN, IC5B.+IN, IC5D.+IN, IN1.GND, IN2.GND
- net N$1: now also IC1G$2.BUF-IN_2, IC1G$2.OUT; no longer U$3G$2.BUF-IN_2, U$3G$2.OUT
- net N$13: now also IC1G$1.BIAS-IN; no longer U$3G$1.BIAS-IN
- net N$15: now also R22.1; no longer R44.1
- net N$16: now also IC1G$2.BUF-OUT_2; no longer U$3G$2.BUF-OUT_2
- net N$17: now also IC1G$1.IN+; no longer U$3G$1.IN+
- net N$18: now also IC3A.-IN; no longer IC5A.-IN
- net N$20: now also IC3C.-IN, IC3C.OUT; no longer IC5C.-IN, IC5C.OUT
- net N$21: now also IC3B.-IN; no longer IC5B.-IN
- net N$22: now also IC1G$2.BIAS-IN; no longer U$3G$2.BIAS-IN
- net N$23: now also IC1G$2.IN+; no longer U$3G$2.IN+
- net N$24: now also IC1G$2.IN-; no longer U$3G$2.IN-
- net N$27: now also IC1G$1.BUF-IN_2, IC1G$1.OUT; no longer U$3G$1.BUF-IN_2, U$3G$1.OUT
- net N$28: now also IC1G$1.BUF-OUT_2; no longer U$3G$1.BUF-OUT_2
- net N$29: now also IC2G$1.IN+; no longer U$4G$1.IN+
- net N$30: now also IC3A.OUT; no longer IC5A.OUT
- net N$31: now also IC2G$2.BIAS-IN; no longer U$4G$2.BIAS-IN
- net N$33: now also IC2G$1.IN-; no longer U$4G$1.IN-
- net N$37: now also IC3D.-IN, IC3D.OUT; no longer IC5D.-IN, IC5D.OUT
- net N$4: now also IC1G$1.IN-; no longer U$3G$1.IN-
- net N$40: now also IC2G$2.IN-; no longer U$4G$2.IN-
- net N$41: now also IC3B.OUT; no longer IC5B.OUT
- net N$43: now also IC2G$2.IN+; no longer U$4G$2.IN+
- net N$44: now also IC2G$1.BUF-OUT_2; no longer U$4G$1.BUF-OUT_2
- net N$46: now also IC2G$2.BUF-OUT_2, IC3C.+IN; no longer IC5C.+IN, U$4G$2.BUF-OUT_2
- net N$5: now also R5.2; no longer R0.2
- net N$55: now also R22.2; no longer R44.2
- net N$57: now also IC2G$1.BUF-IN_2, IC2G$1.OUT; no longer U$4G$1.BUF-IN_2, U$4G$1.OUT
- net N$58: now also IC2G$2.BUF-IN_2, IC2G$2.OUT; no longer U$4G$2.BUF-IN_2, U$4G$2.OUT
- net N$59: now also IC2G$1.BIAS-IN; no longer U$4G$1.BIAS-IN
- net N$6: now also R5.1; no longer R0.1

Commit message: VCF 2.5 beta
VCF Updated to V2.5 14/04/21

Library updated to 3D models.
Changed the CV mixer from Average to Sum and added inverter stage to retain consistency.
Some resistor values reduced to 10K, inline with low noise techniques.
Rerouted and reduced some traces.
Parts:
- added R44: 10k, GMSN:RESISTOR_USR0805
- C4, C5, C6, C7: device GMSN:CAPACITOR-US050-045X075 -> GMSN:CAPACITOR-USC050-045X075
- COF: value 100k -> 10k; device GMSN:RESISTOR_VARIABLE9MM_POT -> GMSN:RESISTOR_VARIABLEPOT_9MM_RED_KNOB
- CV_AT: value 100k -> 10k; device GMSN:RESISTOR_VARIABLE9MM_POT -> GMSN:RESISTOR_VARIABLEPOT_9MM_GREEN_KNOB
- IN1POT, IN1POT1: value 100k -> 10k; device GMSN:RESISTOR_VARIABLE9MM_POT -> GMSN:RESISTOR_VARIABLEPOT_9MM_BLUE_KNOB
- Q: value 100k -> 10k; device GMSN:RESISTOR_VARIABLE9MM_POT -> GMSN:RESISTOR_VARIABLEPOT_9MM_YELLOW_KNOB
- R1, R22, R24, R25, R3, R37, R38, R39, R4, R40, R41, R43: value 100k -> 10k
- R5: device GMSN:RESISTOR_US0204/7 -> GMSN:RESISTOR_US0207/8.5
Connections:
- removed net N$8: IC4D.+IN, R3.2, R4.2
- new net N$34: IC4C.OUT, R1.1, R44.2
- net GND: now also IC4D.+IN; no longer R1.1
- net N$39: now also R3.2, R4.2, R44.1; no longer IC4C.OUT
Other:
- moved on the sheet: COF_CV, IC4C, R21, R3, R4
